Commit message: Tried to build multi grasping pipette

File: pdms_gripper_description/urdf/mycobot_320_pi_2022_workcell_clip.urdf (robot description, URDF)
Before this commit: robot firefighter, 18 links, 17 joints
Links:
- link pipette_holder: geometry collision mesh filename=package://pdms_gripper_description/meshes/pipette_holder_ca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 scale=0.001 0.001 0.001; visual mesh filename=package://pdms_gripper_description/meshes/pipette_holder_ca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
Joints:
- removed joint frame_to_pipette_holder
- removed joint pipette_holder_to_pipette_socket
- added joint frame_to_holder: type fixed, parent frame, child pipette_holder, origin xyz=-0.01413 -0.26972 0.18000 rpy=0.00000 0.00000 1.57080
- added joint holder_to_socket: type fixed, parent pipette_holder, child pipette_socket, origin xyz=0.00000 0.13300 0.00000 rpy=0.00000 0.00000 0.00000

File: pdms_gripper_description/urdf/mycobot_320_pi_2022_workcell_clip_x2.urdf (robot description, URDF)
Before this commit: robot firefighter, 18 links, 17 joints
Links:
- removed link pipette_holder
- removed link pipette_socket
- added link pipette_holder_0; collision mesh filename=package://pdms_gripper_description/meshes/pipette_holder_ca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 scale=0.001 0.001 0.001; visual mesh filename=package://pdms_gripper_description/meshes/pipette_holder_ca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
- added link pipette_holder_1; collision mesh filename=package://pdms_gripper_description/meshes/pipette_holder_ca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 scale=0.001 0.001 0.001; visual mesh filename=package://pdms_gripper_description/meshes/pipette_holder_ca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
- added link pipette_socket_0
- added link pipette_socket_1
Joints:
- removed joint frame_to_pipette_holder
- removed joint pipette_holder_to_pipette_socket
- added joint frame_to_pipette_holder_0: type fixed, parent frame, child pipette_holder_0, origin xyz=-0.01531 -0.34240 0.18000 rpy=0.00000 0.00000 1.43745
- added joint frame_to_pipette_holder_1: type fixed, parent frame, child pipette_holder_1, origin xyz=-0.01531 -0.19704 0.18000 rpy=0.00000 0.00000 1.70415
- added joint pipette_holder_0_to_pipette_socket_0: type fixed, parent pipette_holder_0, child pipette_socket_0, origin xyz=0.00000 0.13300 0.00000 rpy=0.00000 0.00000 0.00000
- added joint pipette_holder_1_to_pipette_socket_1: type fixed, parent pipette_holder_1, child pipette_socket_1, origin xyz=0.00000 0.13300 0.00000 rpy=0.00000 0.00000 0.00000
