Commit message: Add pick-and-place sequence; move frame to arm front; flip pipette upright; single-source pipette pose

File: pdms_gripper_description/urdf/mycobot_320_pi_2022_workcell.urdf (robot description, URDF)
Before this commit: robot firefighter, 18 links, 17 joints
Joints:
- joint frame_to_holder: origin xyz=0.00587 -0.26972 0.25000 rpy=0.00000 0.00000 -1.57080 -> xyz=-0.01413 -0.26972 0.25000 rpy=0.00000 0.00000 1.57080
- joint world_to_frame: origin xyz=0.23913 0.26972 0.00000 rpy=0.00000 0.00000 0.00000 -> xyz=0.26972 -0.34913 0.00000 rpy=0.00000 0.00000 -1.57080

Commit message: Add MoveIt 2 config for 320 workcell; fix collision mesh scale; frame at 410mm standoff

File: pdms_gripper_description/urdf/mycobot_320_pi_2022_workcell.urdf (robot description, URDF)
Before this commit: robot firefighter, 18 links, 17 joints
Links:
- link base: geometry collision mesh filename=package://mycobot_description/urdf/mycobot_320_pi_2022/base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 scale=0.001 0.001 0.001; visual mesh filename=package://mycobot_description/urdf/mycobot_320_pi_2022/base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
- link frame: geometry collision mesh filename=package://pdms_gripper_description/meshes/frame_2020.dae scale=0.001 0.001 0.001; visual mesh filename=package://pdms_gripper_description/meshes/frame_2020.dae
- link gripper_base: geometry collision mesh filename=package://mycobot_description/urdf/pro_adaptive_gripper/gri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 scale=0.001 0.001 0.001; visual mesh filename=package://mycobot_description/urdf/pro_adaptive_gripper/gri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
- link gripper_left1: geometry collision mesh filename=package://pdms_gripper_description/meshes/gripper_left1_for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 scale=0.001 0.001 0.001; visual mesh filename=package://pdms_gripper_description/meshes/gripper_left1_for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
- link gripper_left2: geometry collision mesh filename=package://mycobot_description/urdf/pro_adaptive_gripper/gri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 scale=0.001 0.001 0.001; visual mesh filename=package://mycobot_description/urdf/pro_adaptive_gripper/gri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
- link gripper_left3: geometry collision mesh filename=package://mycobot_description/urdf/pro_adaptive_gripper/gri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 scale=0.001 0.001 0.001; visual mesh filename=package://mycobot_description/urdf/pro_adaptive_gripper/gri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
- link gripper_right1: geometry collision mesh filename=package://pdms_gripper_description/meshes/gripper_right1_fo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 scale=0.001 0.001 0.001; visual mesh filename=package://pdms_gripper_description/meshes/gripper_right1_fo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
- link gripper_right2: geometry collision mesh filename=package://mycobot_description/urdf/pro_adaptive_gripper/gri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 scale=0.001 0.001 0.001; visual mesh filename=package://mycobot_description/urdf/pro_adaptive_gripper/gri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
- link gripper_right3: geometry collision mesh filename=package://mycobot_description/urdf/pro_adaptive_gripper/gri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 scale=0.001 0.001 0.001; visual mesh filename=package://mycobot_description/urdf/pro_adaptive_gripper/gri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
- link link1: geometry collision mesh filename=package://mycobot_description/urdf/mycobot_320_pi_2022/link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 scale=0.001 0.001 0.001; visual mesh filename=package://mycobot_description/urdf/mycobot_320_pi_2022/link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
- link link2: geometry collision mesh filename=package://mycobot_description/urdf/mycobot_320_pi_2022/link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 scale=0.001 0.001 0.001; visual mesh filename=package://mycobot_description/urdf/mycobot_320_pi_2022/link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
- link link3: geometry collision mesh filename=package://mycobot_description/urdf/mycobot_320_pi_2022/link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 scale=0.001 0.001 0.001; visual mesh filename=package://mycobot_description/urdf/mycobot_320_pi_2022/link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
- link link4: geometry collision mesh filename=package://mycobot_description/urdf/mycobot_320_pi_2022/link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 scale=0.001 0.001 0.001; visual mesh filename=package://mycobot_description/urdf/mycobot_320_pi_2022/link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
- link link5: geometry collision mesh filename=package://mycobot_description/urdf/mycobot_320_pi_2022/link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 scale=0.001 0.001 0.001; visual mesh filename=package://mycobot_description/urdf/mycobot_320_pi_2022/link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
- link link6: geometry collision mesh filename=package://mycobot_description/urdf/mycobot_320_pi_2022/link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 scale=0.001 0.001 0.001; visual mesh filename=package://mycobot_description/urdf/mycobot_320_pi_2022/link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
- link pipette_holder: geometry collision mesh filename=package://pdms_gripper_description/meshes/pipette_holder_20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 scale=0.001 0.001 0.001; visual mesh filename=package://pdms_gripper_description/meshes/pipette_holder_20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
Joints:
- joint frame_to_holder: origin xyz=-0.01413 -0.26972 0.25000 rpy=0.00000 0.00000 1.57080 -> xyz=-0.01413 -0.26972 0.18000 rpy=0.00000 0.00000 1.57080
- joint world_to_frame: origin xyz=0.26972 -0.34913 0.00000 rpy=0.00000 0.00000 -1.57080 -> xyz=0.26972 -0.45913 0.00000 rpy=0.00000 0.00000 -1.57080

Commit message: Cantilever holder; capture grasp pose from TF; add home return to sequence

File: pdms_gripper_description/urdf/mycobot_320_pi_2022_workcell.urdf (robot description, URDF)
Before this commit: robot firefighter, 18 links, 17 joints
Joints:
- joint holder_to_socket: origin xyz=0.00000 0.03500 0.00000 rpy=0.00000 0.00000 0.00000 -> xyz=0.00000 0.13300 0.00000 rpy=0.00000 0.00000 0.00000
- joint world_to_frame: origin xyz=0.26972 -0.45913 0.00000 rpy=0.00000 0.00000 -1.57080 -> xyz=0.26972 -0.55713 0.00000 rpy=0.00000 0.00000 -1.57080

Commit message: Cantilever holder; corrected TOOL_OFFSET and gripper travel; head-on grasp; return pipette to holder before release

File: pdms_gripper_description/urdf/mycobot_320_pi_2022_workcell.urdf (robot description, URDF)
Before this commit: robot firefighter, 18 links, 17 joints
Joints:
- removed joint frame_to_pipette_holder
- removed joint pipette_holder_to_pipette_socket
- added joint frame_to_holder: type fixed, parent frame, child pipette_holder, origin xyz=-0.01413 -0.26972 0.18000 rpy=0.00000 0.00000 1.57080
- added joint holder_to_socket: type fixed, parent pipette_holder, child pipette_socket, origin xyz=0.00000 0.13300 0.00000 rpy=0.00000 0.00000 0.00000
